File: sallenkey.kicad_sch (KiCad schematic)
At the start: 44 parts, among them J1 Conn_01x02, J2 Conn_01x03_Pin, J3 Conn_01x05_Pin, U1 LM358, U2 OPA1664

Commit message: Add 2.1 documentation
Other:
- note added: "For 2.1 amplifier filter configuration U2B : Populate R6,R10 Do not populate R12,R18,C14,C16,C19 Connect jumper wire across x1,x2 Summed low output from L_Lo"
- note added: "x1"
- note added: "x2"
Changed lines of the file:
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@@
 	(generator_version "10.0")
 	(paper "A4")
+	(text "x1"
+		(exclude_from_sim no)
+		(at 142.494 99.822 0)
+		(effects
+			(font
+				(size 1.27 1.27)
+			)
+		)
+	)
+	(text "x2"
+		(exclude_from_sim no)
+		(at 142.494 140.716 0)
+		(effects
+			(font
+				(size 1.27 1.27)
+			)
+		)
+	)
+	(text "For 2.1 amplifier filter configuration\nU2B : \n	Populate R6,R10\n	Do not populate R12,R18,C14,C16,C19\nConnect jumper wire across x1,x2\nSummed low output from L_Lo\n"
+		(exclude_from_sim no)
+		(at 180.848 124.968 0)
+		(effects
+			(font
+				(size 1.27 1.27)
+			)
+			(justify left)
+		)
+	)
 	(junction
 		(at 101.6 43.18)
